File: dc31-badge-sao.kicad_pcb (KiCad board)
At the start: 2 copper layers, 40.3 x 92.9 mm, 30 parts, among them J1 Conn_01x03_Pin, U1 ATtiny1616-M

Commit message: added a reset feature
Parts:
- renumbered SWr to SW1
Other:
- board text added: "Nyan"
Changed lines of the file:
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@@
     (property "ki_keywords" "switch single-pole double-throw spdt ON-ON")
     (attr through_hole)
-    (fp_text reference "SWr" (at 5.274213 4.144912 161.701) (layer "B.SilkS")
+    (fp_text reference "SW1" (at 5.274213 4.144912 161.701) (layer "B.SilkS")
         (effects (font (size 1.27 1.27) (thickness 0.254)) (justify mirror))
     )
@@
     (effects (font (size 1 1) (thickness 0.15)) (justify left bottom mirror))
   )
+  (gr_text "Nyan" (at 115.75 63.575 73.2) (layer "B.SilkS")
+    (effects (font (size 1 1) (thickness 0.15)) (justify left bottom mirror))
+  )

Commit message: updates after receiving protos
Parts:
- removed D1: D_Small, Diode_SMD:D_SOD-323
- removed L1: L_Small, Inductor_SMD:L_0805_2012Metric
- removed U2: ~, Package_TO_SOT_SMD:SOT-23-5
- C1: value C_Small -> 0.1 uF
- C2: value C_Small -> 47 uF
- R1: value R_Small -> 100 Ohm
- R2: value R_Small -> 47 Ohm
- moved C2 25.8 mm to (113.5, 130.6)
Connections:
- SW1 pad 1: Net-(D1-A) -> +3.3V
- SW1 pad 3: (no net) -> unconnected-(SW1-C-Pad3)
Routing:
- net Net-(D1-A): track 45.5 -> 0.00 mm
- net +3.3V: track 228.5 -> 213.8 mm, vias 8 -> 9
- net Net-(SW1-C): track 1.75 -> 0.00 mm
