File: dc31-badge-sao.kicad_sch (KiCad schematic)
At the start: 30 parts, among them J1 Conn_01x03_Pin, SW1 SW_SPDT, U1 ATtiny1616-M

Commit message: updates after receiving protos
Connections:
- net at SW1.1 (A): now also L1.1, U2.1 (CE)
- now unconnected: SW1.3 (C)
Changed lines of the file:
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@@
     )
   )
-  (symbol (lib_id "Switch:SW_SPDT") (at 86.36 119.38 0) (unit 1)
-    (in_bom yes) (on_board yes) (dnp no) (fields_autoplaced)
-    (property "Reference" "SW1" (at 86.36 113.4491 0)
+  (symbol (lib_id "Switch:SW_SPDT") (at 86.36 119.38 0) (mirror x) (unit 1)
+    (in_bom yes) (on_board yes) (dnp no)
+    (property "Reference" "SW1" (at 82.55 117.491 0)
       (effects (font (size 1.27 1.27)))
     )
-    (property "Value" "SW_SPDT" (at 86.36 115.3701 0)
+    (property "Value" "SW_SPDT" (at 82.55 115.57 0)
       (effects (font (size 1.27 1.27)))
     )
